Commit message: create metalbot_description, add sdf meshes

File: ros2_ws/src/metalbot/metalbot_description/urdf/metalbot.xacro (robot description, xacro)
@@ -1,8 +1,8 @@
 <?xml version='1.0'?>
-<robot name="rosbot"
+<robot name="metalbot"
   xmlns:xacro="http://www.ros.org/wiki/xacro">
   <xacro:arg name="robot_namespace" default=""/>
   <xacro:property name="namespace" value="$(arg robot_namespace)" />
-  <xacro:include filename="$(find metalbot_gazebo)/urdf/rosbot.gazebo" />
+  <xacro:include filename="$(find metalbot_description)/urdf/metalbot.gazebo" />
   <link name='base_link'>
     <pose>0 0 0.1 0 0 0</pose>
@@ -25,5 +25,5 @@
       <origin xyz="0 0 -0.02" rpy=" 1.5707 0 1.5707"/>
       <geometry>
-        <mesh filename="file://$(find metalbot_gazebo)/meshes/box.dae" scale="0.001 0.001 0.001" />
+        <mesh filename="file://$(find metalbot_description)/meshes/box.dae" scale="0.001 0.001 0.001" />
       </geometry>
     </visual>
@@ -49,5 +49,5 @@
       <origin xyz="0 0 0.055" rpy=" 1.5707 0 1.5707"/>
       <geometry>
-        <mesh filename="file://$(find metalbot_gazebo)/meshes/upper.dae" scale="0.001 0.001 0.001" />
+        <mesh filename="file://$(find metalbot_description)/meshes/upper.dae" scale="0.001 0.001 0.001" />
       </geometry>
     </visual>
@@ -57,5 +57,5 @@
       <origin xyz="0 0 0" rpy="0 0 1.5707"/>
       <geometry>
-        <mesh filename="file://$(find metalbot_gazebo)/meshes/wheel-v2.stl" scale="0.001 0.001 0.001" />
+        <mesh filename="file://$(find metalbot_description)/meshes/wheel-v2.stl" scale="0.001 0.001 0.001" />
       </geometry>
       <surface>
@@ -71,5 +71,5 @@
       <origin xyz="0 0 0" rpy="0 0 1.5707"/>
       <geometry>
-        <mesh filename="file://$(find metalbot_gazebo)/meshes/wheel.dae" scale="0.001 0.001 0.001" />
+        <mesh filename="file://$(find metalbot_description)/meshes/wheel.dae" scale="0.001 0.001 0.001" />
       </geometry>
     </visual>
@@ -87,5 +87,5 @@
       <origin xyz="0 0 0" rpy="0 0 -1.5707"/>
       <geometry>
-        <mesh filename="file://$(find metalbot_gazebo)/meshes/wheel-v2.stl" scale="0.001 0.001 0.001" />
+        <mesh filename="file://$(find metalbot_description)/meshes/wheel-v2.stl" scale="0.001 0.001 0.001" />
       </geometry>
       <surface>
@@ -101,5 +101,5 @@
       <origin xyz="0 0 0" rpy="0 0 -1.5707"/>
       <geometry>
-        <mesh filename="file://$(find metalbot_gazebo)/meshes/wheel.dae" scale="0.001 0.001 0.001" />
+        <mesh filename="file://$(find metalbot_description)/meshes/wheel.dae" scale="0.001 0.001 0.001" />
       </geometry>
     </visual>
@@ -117,5 +117,5 @@
       <origin xyz="0 0 0" rpy="0 0 1.5707"/>
       <geometry>
-        <mesh filename="file://$(find metalbot_gazebo)/meshes/wheel-v2.stl" scale="0.001 0.001 0.001" />
+        <mesh filename="file://$(find metalbot_description)/meshes/wheel-v2.stl" scale="0.001 0.001 0.001" />
       </geometry>
       <surface>
@@ -131,5 +131,5 @@
       <origin xyz="0 0 0" rpy="0 0 1.5707"/>
       <geometry>
-        <mesh filename="file://$(find metalbot_gazebo)/meshes/wheel.dae" scale="0.001 0.001 0.001" />
+        <mesh filename="file://$(find metalbot_description)/meshes/wheel.dae" scale="0.001 0.001 0.001" />
       </geometry>
     </visual>
@@ -147,5 +147,5 @@
       <origin xyz="0 0 0" rpy="0 0 -1.5707"/>
       <geometry>
-        <mesh filename="file://$(find metalbot_gazebo)/meshes/wheel-v2.stl" scale="0.001 0.001 0.001" />
+        <mesh filename="file://$(find metalbot_description)/meshes/wheel-v2.stl" scale="0.001 0.001 0.001" />
       </geometry>
       <surface>
@@ -161,5 +161,5 @@
       <origin xyz="0 0 0" rpy="0 0 -1.5707"/>
       <geometry>
-        <mesh filename="file://$(find metalbot_gazebo)/meshes/wheel.dae" scale="0.001 0.001 0.001" />
+        <mesh filename="file://$(find metalbot_description)/meshes/wheel.dae" scale="0.001 0.001 0.001" />
       </geometry>
     </visual>
@@ -258,5 +258,5 @@
       <origin xyz="-0.01 0 -0.03" rpy="1.5707 0 1.5707"/>
       <geometry>
-        <mesh filename="file://$(find metalbot_gazebo)/meshes/astra.dae" scale="0.001 0.001 0.001" />
+        <mesh filename="file://$(find metalbot_description)/meshes/astra.dae" scale="0.001 0.001 0.001" />
       </geometry>
     </visual>

Commit message: rbp, separeate configs

File: ros2_ws/src/metalbot/metalbot_description/urdf/metalbot.xacro (robot description, xacro)
@@ -244,5 +244,5 @@
   <joint name="astra_joint" type="fixed">
     <axis xyz="0 0 0" />
-    <origin xyz="-0.03 0 0.18" rpy="0 0 0"/>
+    <origin xyz="0.16 0 0.18" rpy="0 0 0"/>
     <parent link="base_link"/>
     <child link="camera_link"/>

Commit message: add urdf to t265, d455

File: ros2_ws/src/metalbot/metalbot_description/urdf/metalbot.xacro (robot description, xacro)
@@ -248,4 +248,28 @@
     <child link="camera_link"/>
   </joint>
+  <joint name="camera_link_to_depth" type="fixed">
+    <axis xyz="0 0 0" />
+    <origin xyz="0 -0.05 0" rpy="0 0 0"/>
+    <parent link="camera_link"/>
+    <child link="camera_aligned_depth_to_color"/>
+  </joint>
+  <joint name="depth_to_optical" type="fixed">
+    <axis xyz="0 0 0" />
+    <origin xyz="0 0 0" rpy="-1.57 0 -1.57"/>
+    <parent link="camera_aligned_depth_to_color"/>
+    <child link="camera_color_optical_frame"/>
+  </joint>
+  <joint name="camera_pose_to_base_link" type="fixed">
+    <axis xyz="0 0 0" />
+    <origin xyz="-0.14 -0.01 -0.215" rpy="0 0 0"/>
+    <parent link="camera_pose_frame"/>
+    <child link="base_link"/>
+  </joint>
+  <link name="camera_aligned_depth_to_color">
+  </link>
+  <link name="camera_pose_frame">
+  </link>
+  <link name="camera_color_optical_frame">
+  </link>
   <link name="camera_link">
     <collision>
